File: Hardware/MAVRIC-Main.sch (KiCad schematic (older format))
At the start: 0 parts

Commit message: Add basic connector and ChipKit headers
Parts:
- added J1: MTR1, ~, symbol CONN-8
- added J10: CAM, ~, symbol CONN-8
- added J11: CK-PWR, ~, symbol CONN-6
- added J12: CK-A0, ~, symbol CONN-8
- added J13: CK-A1, ~, symbol CONN-8
- added J14: CK-COM, ~, symbol CONN-8
- added J15: CK-D0, ~, symbol CONN-8X2
- added J16: CK-X0, ~, symbol CONN-8X2
- added J17: CK-D1, ~, symbol CONN-8X2
- added J18: CK-X1, ~, symbol CONN-8X2
- added J2: MTR4, ~, symbol CONN-8
- added J3: MTR2, ~, symbol CONN-8
- added J4: MTR5, ~, symbol CONN-8
- added J5: MTR3, ~, symbol CONN-8
- added J6: MTR6, ~, symbol CONN-8
- added J7: VID, ~, symbol CONN-8
- added J8: DAT, ~, symbol CONN-8
- added J9: ARM, ~, symbol CONN-8
Connections:
- net labels added: +3.3V, +5V, +BATT, A0, A1, A10, A11, A12, A13, A14, A15, A2, A3, A4, A5, A6, A7, A8, A9, ARef, CK10, CK11, CK12, CK13, CK2, CK22, CK23, CK24, CK25, CK26, CK27, CK28, CK29, CK3, CK30, CK31, CK32, CK33, CK34, CK35, CK36, CK37, CK38, CK39, CK4, CK40, CK41, CK42, CK43, CK44, CK45, CK46, CK47, CK48, CK49, CK5, CK50, CK51, CK52, CK53, CK6, CK7, CK70, CK71, CK72, CK73, CK74, CK75, CK76, CK77, CK78, CK79, CK8, CK80, CK81, CK82, CK83, CK84, CK85, CK9, GND, RST, RX0, RX1, RX2, RX3, SCL, SDA, TX0, TX1, TX2, TX3
- wire segments 0 -> 99

Commit message: Replace arm and camera connectors with vertical style
Other:
- moved on the sheet: J11
Changed lines of the file:
@@
 L CONN-6 J11
 U 1 1 522BA607
-P 4300 1250
-F 0 "J11" H 4300 1600 60  0000 C CNN
-F 1 "CK-PWR" H 4300 900 60  0000 C CNN
-F 2 "~" H 4300 1250 60  0000 C CNN
-F 3 "~" H 4300 1250 60  0000 C CNN
-	1    4300 1250
+P 10000 4250
+F 0 "J11" H 10000 4600 60  0000 C CNN
+F 1 "CK-PWR" H 10000 3900 60  0000 C CNN
+F 2 "~" H 10000 4250 60  0000 C CNN
+F 3 "~" H 10000 4250 60  0000 C CNN
+	1    10000 4250
 	1    0    0    -1
 $EndComp
@@
 	1    0    0    -1
 $EndComp
-Text Label 5300 1000 0    60   ~ 0
+Text Label 11000 4000 0    60   ~ 0
 RST
 $Comp
 L +3.3V #PWR01
 U 1 1 522BAE22
-P 4800 900
-F 0 "#PWR01" H 4800 860 30  0001 C CNN
-F 1 "+3.3V" H 4800 1010 30  0000 C CNN
-F 2 "" H 4800 900 60  0000 C CNN
-F 3 "" H 4800 900 60  0000 C CNN
-	1    4800 900
+P 10500 3900
+F 0 "#PWR01" H 10500 3860 30  0001 C CNN
+F 1 "+3.3V" H 10500 4010 30  0000 C CNN
+F 2 "" H 10500 3900 60  0000 C CNN
+F 3 "" H 10500 3900 60  0000 C CNN
+	1    10500 3900
 	1    0    0    -1
 $EndComp
@@
 L +5V #PWR02
 U 1 1 522BAE3B
-P 5000 900
-F 0 "#PWR02" H 5000 990 20  0001 C CNN
-F 1 "+5V" H 5000 990 30  0000 C CNN
-F 2 "" H 5000 900 60  0000 C CNN
-F 3 "" H 5000 900 60  0000 C CNN
-	1    5000 900
+P 10700 3900
+F 0 "#PWR02" H 10700 3990 20  0001 C CNN
+F 1 "+5V" H 10700 3990 30  0000 C CNN
+F 2 "" H 10700 3900 60  0000 C CNN
+F 3 "" H 10700 3900 60  0000 C CNN
+	1    10700 3900
 	1    0    0    -1
 $EndComp
@@
 L +BATT #PWR03
 U 1 1 522BAE4C
-P 5200 900
-F 0 "#PWR03" H 5200 850 20  0001 C CNN
-F 1 "+BATT" H 5200 1000 30  0000 C CNN
-F 2 "" H 5200 900 60  0000 C CNN
-F 3 "" H 5200 900 60  0000 C CNN
-	1    5200 900
+P 10900 3900
+F 0 "#PWR03" H 10900 3850 20  0001 C CNN
+F 1 "+BATT" H 10900 4000 30  0000 C CNN
+F 2 "" H 10900 3900 60  0000 C CNN
+F 3 "" H 10900 3900 60  0000 C CNN
+	1    10900 3900
 	1    0    0    -1
 $EndComp
@@
 L GND #PWR04
 U 1 1 522BAE5D
-P 4800 1600
-F 0 "#PWR04" H 4800 1600 30  0001 C CNN
-F 1 "GND" H 4800 1530 30  0001 C CNN
-F 2 "" H 4800 1600 60  0000 C CNN
-F 3 "" H 4800 1600 60  0000 C CNN
-	1    4800 1600
+P 10500 4600
+F 0 "#PWR04" H 10500 4600 30  0001 C CNN
+F 1 "GND" H 10500 4530 30  0001 C CNN
+F 2 "" H 10500 4600 60  0000 C CNN
+F 3 "" H 10500 4600 60  0000 C CNN
+	1    10500 4600
 	1    0    0    -1
 $EndComp
@@
 $EndComp
 Wire Wire Line
-	4800 1600 4800 1300
-Wire Wire Line
-	4800 1300 4700 1300
-Wire Wire Line
-	4700 1400 4800 1400
-Connection ~ 4800 1400
-Wire Wire Line
-	4700 1500 5200 1500
-Wire Wire Line
-	5200 1500 5200 900
-Wire Wire Line
-	4700 1000 5300 1000
-Wire Wire Line
-	4700 1100 4800 1100
-Wire Wire Line
-	4800 1100 4800 900
-Wire Wire Line
-	4700 1200 5000 1200
-Wire Wire Line
-	5000 1200 5000 900
+	10500 4600 10500 4300
+Wire Wire Line
+	10500 4300 10400 4300
+Wire Wire Line
+	10400 4400 10500 4400
+Connection ~ 10500 4400
+Wire Wire Line
+	10400 4500 10900 4500
+Wire Wire Line
+	10900 4500 10900 3900
+Wire Wire Line
+	10400 4000 11000 4000
+Wire Wire Line
+	10400 4100 10500 4100
+Wire Wire Line
+	10500 4100 10500 3900
+Wire Wire Line
+	10400 4200 10700 4200
+Wire Wire Line
+	10700 4200 10700 3900
 Wire Wire Line
 	8500 700  8600 700

Commit message: Swap vid/agnd to comply with camera change
Parts:
- added J19: GPS, ~, symbol CONN-8
- added U1: SN74LVC1G125, ~, symbol SN74LVC1G125
Connections:
- net labels added: CamGnd, CamPwr, MotorTx, TxGnd, TxPwr, VidGnd, Video
- wire segments 99 -> 136
- no-connect marks 0 -> 5
Other:
- moved on the sheet: J1, J10, J2, J3, J4, J5, J6, J7, J8, J9

Commit message: Rough pin out of most systems
Parts:
- added C1: 0.1uF, ~, symbol C
- added J20: CONN-DC, ~, symbol CONN-DC
Connections:
- net labels added: Dir1, Dir2, Dir3, Dir4, Dir5, Dir6, En1, En2, En3, En4, En5, En6, Mtr1, Mtr2, Mtr3, Mtr4, Mtr5, Mtr6, Step1, Step2, Step3, Step4, Step5, Step6
- net labels removed: CamGnd, CamPwr, TxGnd, TxPwr
- wire segments 136 -> 207
- no-connect marks 5 -> 4

Commit message: Finish 1v0 circuit board!
Parts:
- added C2: 0.1uF, ~, symbol C
- added D1: LED, ~, symbol LED
- added R1: 36k, ~, symbol R
- added R2: 10k, ~, symbol R
- added R3: R, ~, symbol R
Connections:
- net labels added: FB1, FB2, FB3, FB4, FB5, FB6
- wire segments 207 -> 221
Other:
- moved on the sheet: J20
Changed lines of the file:
@@
 Sheet 1 1
 Title ""
-Date "9 sep 2013"
+Date "12 sep 2013"
 Rev ""
 Comp ""
@@
 Text Label 9000 6100 2    60   ~ 0
 TX1
-Text Label 3300 1000 0    60   ~ 0
-TX2
+Text Label 3400 1000 0    60   ~ 0
+RX2
 Text Label 3400 2200 0    60   ~ 0
 TX3
 Text Label 3500 5600 0    60   ~ 0
 RX1
-Text Label 3300 800  0    60   ~ 0
-RX2
+Text Label 3400 800  0    60   ~ 0
+TX2
 Text Label 3400 2500 0    60   ~ 0
 RX3
@@
 Text Label 3400 2100 0    60   ~ 0
 Video
-Text Label 3400 4400 0    60   ~ 0
+Text Label 3400 4500 0    60   ~ 0
 Video
 NoConn ~ 3200 4600
@@
 Text Label 3400 2000 0    60   ~ 0
 VidGnd
-Text Label 3400 4500 0    60   ~ 0
+Text Label 3400 4400 0    60   ~ 0
 VidGnd
 $Comp
@@
 NoConn ~ 3200 6100
 Text Label 1600 1400 0    60   ~ 0
-A1
+FB1
 Text Label 1600 2600 0    60   ~ 0
-A2
+FB2
 Text Label 1600 3800 0    60   ~ 0
-A3
+FB3
 Text Label 1600 5000 0    60   ~ 0
-A4
+FB4
 Text Label 1600 6200 0    60   ~ 0
-A5
+FB5
 Text Label 1600 7400 0    60   ~ 0
-A6
+FB6
 $Comp
 L +BATT #PWR08
@@
 L CONN-DC J20
 U 1 1 522E4D58
-P 5600 1050
-F 0 "J20" H 5600 1200 60  0000 C CNN
-F 1 "CONN-DC" H 5600 900 60  0000 C CNN
-F 2 "~" H 5600 1050 60  0000 C CNN
-F 3 "~" H 5600 1050 60  0000 C CNN
-	1    5600 1050
+P 4700 1050
+F 0 "J20" H 4700 1200 60  0000 C CNN
+F 1 "CONN-DC" H 4700 900 60  0000 C CNN
+F 2 "~" H 4700 1050 60  0000 C CNN
+F 3 "~" H 4700 1050 60  0000 C CNN
+	1    4700 1050
 	1    0    0    -1
 $EndComp
@@
 L GND #PWR014
 U 1 1 522E4D67
-P 6000 1200
-F 0 "#PWR014" H 6000 1200 30  0001 C CNN
-F 1 "GND" H 6000 1130 30  0001 C CNN
-F 2 "" H 6000 1200 60  0000 C CNN
-F 3 "" H 6000 1200 60  0000 C CNN
-	1    6000 1200
+P 5100 1200
+F 0 "#PWR014" H 5100 1200 30  0001 C CNN
+F 1 "GND" H 5100 1130 30  0001 C CNN
+F 2 "" H 5100 1200 60  0000 C CNN
+F 3 "" H 5100 1200 60  0000 C CNN
+	1    5100 1200
 	1    0    0    -1
 $EndComp
@@
 L +BATT #PWR015
 U 1 1 522E4D76
-P 6000 900
-F 0 "#PWR015" H 6000 850 20  0001 C CNN
-F 1 "+BATT" H 6000 1000 30  0000 C CNN
-F 2 "" H 6000 900 60  0000 C CNN
-F 3 "" H 6000 900 60  0000 C CNN
-	1    6000 900
+P 5100 900
+F 0 "#PWR015" H 5100 850 20  0001 C CNN
+F 1 "+BATT" H 5100 1000 30  0000 C CNN
+F 2 "" H 5100 900 60  0000 C CNN
+F 3 "" H 5100 900 60  0000 C CNN
+	1    5100 900
 	1    0    0    -1
 $EndComp
@@
 Connection ~ 3300 2700
 Wire Wire Line
-	6000 900  6000 1000
-Wire Wire Line
-	6000 1000 5900 1000
-Wire Wire Line
-	5900 1100 6000 1100
-Wire Wire Line
-	6000 1100 6000 1200
+	5100 900  5100 1000
+Wire Wire Line
+	5100 1000 5000 1000
+Wire Wire Line
+	5000 1100 5100 1100
+Wire Wire Line
+	5100 1100 5100 1200
 Wire Wire Line
 	9700 5500 9700 5700
@@
 	1500 1500 1500 1600
 Wire Wire Line
-	1400 1400 1600 1400
-Wire Wire Line
-	1400 2600 1600 2600
+	1400 1400 1900 1400
+Wire Wire Line
+	1400 2600 1900 2600
 Wire Wire Line
 	1400 2700 1500 2700
@@
 	1500 2700 1500 2800
 Wire Wire Line
-	1400 3800 1600 3800
+	1400 3800 1900 3800
 Wire Wire Line
 	1400 3900 1500 3900
@@
 	1500 3900 1500 4000
 Wire Wire Line
-	1400 5000 1900 5000
-Wire Wire Line
 	1400 5100 1500 5100
 Wire Wire Line
 	1500 5100 1500 5200
 Wire Wire Line
-	1400 6200 1600 6200
+	1400 6200 1900 6200
 Wire Wire Line
 	1400 6300 1500 6300
@@
 	1500 6300 1500 6400
 Wire Wire Line
-	1400 7400 1600 7400
+	1400 7400 1900 7400
 Wire Wire Line
 	1400 7500 1500 7500
@@
 	1400 4500 1900 4500
 Wire Wire Line
-	1400 4700 1600 4700
+	1400 4700 1900 4700
 Wire Wire Line
 	1400 4800 1900 4800
@@
 Wire Wire Line
 	1400 7300 1900 7300
-Text Label 1900 5000 0    60   ~ 0
+Text Label 1900 4900 0    60   ~ 0
 CK13
-Text Label 1900 4900 0    60   ~ 0
+Text Label 1900 4800 0    60   ~ 0
 CK12
-Text Label 1900 4800 0    60   ~ 0
+Text Label 1900 4700 0    60   ~ 0
 CK11
 Text Label 1900 6100 0    60   ~ 0
@@
 CK81
 Text Label 1900 3700 0    60   ~ 0
+CK71
+Text Label 1900 3600 0    60   ~ 0
+CK72
+Text Label 1900 3500 0    60   ~ 0
+CK73
+Text Label 1900 3300 0    60   ~ 0
 CK74
-Text Label 1900 3600 0    60   ~ 0
-CK75
-Text Label 1900 3500 0    60   ~ 0
-CK76
-Text Label 1900 3300 0    60   ~ 0
-CK77
 Wire Wire Line
 	3200 5700 3300 5700
 Connection ~ 3300 6200
+Wire Wire Line
+	3400 800  3200 800
+Wire Wire Line
+	3400 1000 3200 1000
+$Comp
+L GND #PWR031
+U 1 1 522FF35C
+P 3300 1600
+F 0 "#PWR031" H 3300 1600 30  0001 C CNN
+F 1 "GND" H 3300 1530 30  0001 C CNN
+F 2 "" H 3300 1600 60  0000 C CNN
+F 3 "" H 3300 1600 60  0000 C CNN
+	1    3300 1600
+	1    0    0    -1
+$EndComp
+Wire Wire Line
+	3300 1600 3300 900
+Wire Wire Line
+	3300 900  3200 900
+Wire Wire Line
+	3200 1300 3300 1300
+Connection ~ 3300 1300
+Wire Wire Line
+	1400 5000 1900 5000
+$Comp
+L R R1
+U 1 1 5230F099
+P 6700 1150
+F 0 "R1" H 6700 1250 60  0000 C CNN
+F 1 "36k" H 6700 1150 60  0000 C CNN
+F 2 "~" H 6700 1150 60  0000 C CNN
+F 3 "~" H 6700 1150 60  0000 C CNN
+	1    6700 1150
+	0    -1   -1   0
+$EndComp
+$Comp
+L R R2
+U 1 1 5230F0A8
+P 6700 1850
+F 0 "R2" H 6700 1950 60  0000 C CNN
+F 1 "10k" H 6700 1850 60  0000 C CNN
+F 2 "~" H 6700 1850 60  0000 C CNN
+F 3 "~" H 6700 1850 60  0000 C CNN
+	1    6700 1850
+	0    -1   -1   0
+$EndComp
+$Comp
+L C C2
+U 1 1 5230F0B7
+P 7000 1850
+F 0 "C2" H 7050 2000 60  0000 L CNN
+F 1 "0.1uF" H 7050 1700 60  0000 L CNN
+F 2 "~" H 7000 1850 60  0000 C CNN
+F 3 "~" H 7000 1850 60  0000 C CNN
+	1    7000 1850
+	1    0    0    -1
+$EndComp
+Text Label 7100 1500 0    60   ~ 0
+A0
+$Comp
+L GND #PWR032
+U 1 1 5230F0C6
+P 6700 2200
+F 0 "#PWR032" H 6700 2200 30  0001 C CNN
+F 1 "GND" H 6700 2130 30  0001 C CNN
+F 2 "" H 6700 2200 60  0000 C CNN
+F 3 "" H 6700 2200 60  0000 C CNN
+	1    6700 2200
+	1    0    0    -1
+$EndComp
+$Comp
+L GND #PWR033
+U 1 1 5230F0D5
+P 7000 2200
+F 0 "#PWR033" H 7000 2200 30  0001 C CNN
+F 1 "GND" H 7000 2130 30  0001 C CNN
+F 2 "" H 7000 2200 60  0000 C CNN
+F 3 "" H 7000 2200 60  0000 C CNN
+	1    7000 2200
+	1    0    0    -1
+$EndComp
+$Comp
+L +BATT #PWR034
+U 1 1 5230F0E4
+P 6700 800
+F 0 "#PWR034" H 6700 750 20  0001 C CNN
+F 1 "+BATT" H 6700 900 30  0000 C CNN
+F 2 "" H 6700 800 60  0000 C CNN
+F 3 "" H 6700 800 60  0000 C CNN
+	1    6700 800
+	1    0    0    -1
+$EndComp
+Wire Wire Line
+	6700 800  6700 900
+Wire Wire Line
+	6700 1400 6700 1600
+Wire Wire Line
+	6700 2100 6700 2200
+Wire Wire Line
+	6700 1500 7100 1500
+Connection ~ 6700 1500
+Wire Wire Line
+	7000 1600 7000 1500
+Connection ~ 7000 1500
+Wire Wire Line
+	7000 2100 7000 2200
+$Comp
+L LED D1
+U 1 1 5230F72D
+P 6300 1850
+F 0 "D1" H 6300 1975 60  0000 C CNN
+F 1 "LED" H 6300 1750 60  0000 C CNN
+F 2 "~" H 6300 1850 60  0000 C CNN
+F 3 "~" H 6300 1850 60  0000 C CNN
+	1    6300 1850
+	0    -1   -1   0
+$EndComp
+$Comp
+L R R3
+U 1 1 5230F73C
+P 6300 1150
+F 0 "R3" H 6300 1250 60  0000 C CNN
+F 1 "R" H 6300 1150 60  0000 C CNN
+F 2 "~" H 6300 1150 60  0000 C CNN
+F 3 "~" H 6300 1150 60  0000 C CNN
+	1    6300 1150
+	0    -1   -1   0
+$EndComp
+$Comp
+L +BATT #PWR035
+U 1 1 5230F74B
+P 6300 800
+F 0 "#PWR035" H 6300 750 20  0001 C CNN
+F 1 "+BATT" H 6300 900 30  0000 C CNN
+F 2 "" H 6300 800 60  0000 C CNN
+F 3 "" H 6300 800 60  0000 C CNN
+	1    6300 800
+	1    0    0    -1
+$EndComp
+$Comp
+L GND #PWR036
+U 1 1 5230F934
+P 6300 2200
+F 0 "#PWR036" H 6300 2200 30  0001 C CNN
+F 1 "GND" H 6300 2130 30  0001 C CNN
+F 2 "" H 6300 2200 60  0000 C CNN
+F 3 "" H 6300 2200 60  0000 C CNN
+	1    6300 2200
+	1    0    0    -1
+$EndComp
+Wire Wire Line
+	6300 800  6300 900
+Wire Wire Line
+	6300 1400 6300 1600
+Wire Wire Line
+	6300 2100 6300 2200
+Text Label 1900 1400 0    60   ~ 0
+A2
+Text Label 1900 2600 0    60   ~ 0
+A4
+Text Label 1900 3800 0    60   ~ 0
+A6
+Text Label 1900 5000 0    60   ~ 0
+A1
+Text Label 1900 6200 0    60   ~ 0
+A3
+Text Label 1900 7400 0    60   ~ 0
+A5
 $EndSCHEMATC

Commit message: Add some bom values
Parts:
- U1: Distributor Part No (none) -> 296-11604-1-ND
Changed lines of the file:
@@
 Sheet 1 1
 Title ""
-Date "12 sep 2013"
+Date "24 sep 2013"
 Rev ""
 Comp ""
@@
 F 2 "~" H 9700 6100 60  0000 C CNN
 F 3 "~" H 9700 6100 60  0000 C CNN
+F 4 "296-11604-1-ND" H 9700 6100 60  0001 C CNN "Distributor Part No"
 	1    9700 6100
 	1    0    0    -1
