File: Hardware/$Regulator +3v3.sch (KiCad schematic (older format))
At the start: 22 parts, among them U3 AOZ1280CI, U4 AP65552SP-13

Commit message: PCB Almost Complete
Parts:
- C24: renamed from C?; footprint (none) -> Capacitors_SMD:C_1206_HandSoldering
Changed lines of the file:
@@
 $EndComp
 $Comp
-L Capacitor C?
+L Capacitor C24
 U 1 1 5548FC27
 P 3750 3100
-F 0 "C?" V 3600 3200 60  0000 L CNN
+F 0 "C24" V 3600 3200 60  0000 L CNN
 F 1 "4.7uF" V 3700 3200 60  0000 L CNN
-F 2 "" H 3650 3100 60  0001 C CNN
+F 2 "Capacitors_SMD:C_1206_HandSoldering" H 3650 3100 60  0001 C CNN
 F 3 "" H 3750 3200 60  0001 C CNN
 F 4 "Value" H 3750 3100 60  0001 C CNN "Manufacturer"
@@
 $EndComp
 $Comp
-L GND #PWR?
+L GND #PWR026
 U 1 1 5548FCC9
 P 3750 3400
-F 0 "#PWR?" H 3750 3150 60  0001 C CNN
+F 0 "#PWR026" H 3750 3150 60  0001 C CNN
 F 1 "GND" H 3750 3250 60  0000 C CNN
 F 2 "" H 3750 3400 60  0000 C CNN
